File: Electricals/Examples/[DFR1142]Lite Carrier for LattePanda Mu/PSU.kicad_sch (KiCad schematic)
At the start: 87 parts, among them J17 Barrel_Jack_Switch, J18 USB_C_Receptacle_USB2.0, Q5 2N7002, Q6 2N7002, Q7 NCE30P28Q, Q8 2N7002, SW1 SW_Push, SW2 SW_Push, U13 TL431DBZ, U14 CH224K, U15 SY8253ADC, U16 SY8253ADC

Commit message: new format
Changed lines of the file:
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@@
 (kicad_sch
-	(version 20231120)
+	(version 20250114)
 	(generator "eeschema")
-	(generator_version "8.0")
+	(generator_version "9.0")
 	(paper "A2")
 	(title_block
@@
 		(company "DFRobot")
 	)
+	(text "soft start"
+		(exclude_from_sim no)
+		(at 288.29 105.41 0)
+		(effects
+			(font
+				(size 1.27 1.27)
+			)
+			(justify left bottom)
+		)
+	)
+	(text "15V PD Input"
+		(exclude_from_sim no)
+		(at 162.56 237.49 0)
+		(effects
+			(font
+				(size 2.54 2.54)
+				(thickness 0.508)
+				(bold yes)
+			)
+			(justify left bottom)
+		)
+	)
+	(text "SY8253ADC 23V 3A 500kHz\n"
+		(exclude_from_sim no)
+		(at 372.11 152.4 0)
+		(effects
+			(font
+				(size 2.54 2.54)
+				(thickness 0.508)
+				(bold yes)
+			)
+			(justify left bottom)
+		)
+	)
+	(text "LattePanda Mu has integrated pull-up resistors."
+		(exclude_from_sim no)
+		(at 393.7 292.1 0)
+		(effects
+			(font
+				(size 1.27 1.27)
+			)
+			(justify left)
+		)
+	)
+	(text "Power for PCIe x4 OVP@13.86V"
+		(exclude_from_sim no)
+		(at 232.41 87.63 0)
+		(effects
+			(font
+				(size 2 2)
+				(thickness 0.2794)
+				(bold yes)
+			)
+			(justify left bottom)
+		)
+	)
+	(text "Vout=0.6*(75+10)/10=5.1V"
+		(exclude_from_sim no)
+		(at 420.37 157.48 0)
+		(effects
+			(font
+				(size 1.397 1.397)
+				(thickness 0.2794)
+				(bold yes)
+			)
+			(justify left bottom)
+		)
+	)
+	(text "12V DC Input(12V 6A-10A)"
+		(exclude_from_sim no)
+		(at 162.56 152.4 0)
+		(effects
+			(font
+				(size 2.54 2.54)
+				(thickness 0.508)
+				(bold yes)
+			)
+			(justify left bottom)
+		)
+	)
+	(text "CH224K get DC 15V power from USB-PD adapter"
+		(exclude_from_sim no)
+		(at 245.11 276.86 0)
+		(effects
+			(font
+				(size 1.397 1.397)
+				(thickness 0.2794)
+				(bold yes)
+			)
+			(justify left bottom)
+		)
+	)
+	(text "PCIe Power Enable LED"
+		(exclude_from_sim no)
+		(at 387.35 107.95 0)
+		(effects
+			(font
+				(size 1.27 1.27)
+			)
+			(justify left)
+		)
+	)
+	(text "Pullup power for bios_sel\n"
+		(exclude_from_sim no)
+		(at 400.05 133.35 0)
+		(effects
+			(font
+				(size 2 2)
+				(thickness 0.2794)
+				(bold yes)
+			)
+			(justify left bottom)
+		)
+	)
+	(text "Vout=0.6*(21.5+4.7)/4.7=3.446V"
+		(exclude_from_sim no)
+		(at 420.37 195.58 0)
+		(effects
+			(font
+				(size 1.397 1.397)
+				(thickness 0.2794)
+				(bold yes)
+			)
+			(justify left bottom)
+		)
+	)
 	(junction
 		(at 283.21 147.32)
@@
 		)
 	)
-	(text "soft start"
-		(exclude_from_sim no)
-		(at 288.29 105.41 0)
-		(effects
-			(font
-				(size 1.27 1.27)
-			)
-			(justify left bottom)
-		)
-	)
-	(text "15V PD Input"
-		(exclude_from_sim no)
-		(at 162.56 237.49 0)
-		(effects
-			(font
-				(size 2.54 2.54)
-				(thickness 0.508)
-				(bold yes)
-			)
-			(justify left bottom)
-		)
-	)
-	(text "SY8253ADC 23V 3A 500kHz\n"
-		(exclude_from_sim no)
-		(at 372.11 152.4 0)
-		(effects
-			(font
-				(size 2.54 2.54)
-				(thickness 0.508)
-				(bold yes)
-			)
-			(justify left bottom)
-		)
-	)
-	(text "LattePanda Mu has integrated pull-up resistors."
-		(exclude_from_sim no)
-		(at 393.7 292.1 0)
-		(effects
-			(font
-				(size 1.27 1.27)
-			)
-			(justify left)
-		)
-	)
-	(text "Power for PCIe x4 OVP@13.86V"
-		(exclude_from_sim no)
-		(at 232.41 87.63 0)
-		(effects
-			(font
-				(size 2 2)
-				(thickness 0.2794)
-				(bold yes)
-			)
-			(justify left bottom)
-		)
-	)
-	(text "Vout=0.6*(75+10)/10=5.1V"
-		(exclude_from_sim no)
-		(at 420.37 157.48 0)
-		(effects
-			(font
-				(size 1.397 1.397)
-				(thickness 0.2794)
-				(bold yes)
-			)
-			(justify left bottom)
-		)
-	)
-	(text "12V DC Input(12V 6A-10A)"
-		(exclude_from_sim no)
-		(at 162.56 152.4 0)
-		(effects
-			(font
-				(size 2.54 2.54)
-				(thickness 0.508)
-				(bold yes)
-			)
-			(justify left bottom)
-		)
-	)
-	(text "CH224K get DC 15V power from USB-PD adapter"
-		(exclude_from_sim no)
-		(at 245.11 276.86 0)
-		(effects
-			(font
-				(size 1.397 1.397)
-				(thickness 0.2794)
-				(bold yes)
-			)
-			(justify left bottom)
-		)
-	)
-	(text "PCIe Power Enable LED"
-		(exclude_from_sim no)
-		(at 387.35 107.95 0)
-		(effects
-			(font
-				(size 1.27 1.27)
-			)
-			(justify left)
-		)
-	)
-	(text "Pullup power for bios_sel\n"
-		(exclude_from_sim no)
-		(at 400.05 133.35 0)
-		(effects
-			(font
-				(size 2 2)
-				(thickness 0.2794)
-				(bold yes)
-			)
-			(justify left bottom)
-		)
-	)
-	(text "Vout=0.6*(21.5+4.7)/4.7=3.446V"
-		(exclude_from_sim no)
-		(at 420.37 195.58 0)
-		(effects
-			(font
-				(size 1.397 1.397)
-				(thickness 0.2794)
-				(bold yes)
-			)
-			(justify left bottom)
-		)
-	)
 	(label "PWR_EN"
 		(at 306.07 137.16 0)
-		(fields_autoplaced yes)
 		(effects
 			(font
@@
 	(label "PWR_EN"
 		(at 361.95 207.01 0)
-		(fields_autoplaced yes)
 		(effects
 			(font
@@
 	(label "PWR_C_D+"
 		(at 189.23 264.16 0)
-		(fields_autoplaced yes)
 		(effects
 			(font
@@
 	(label "CC2"
 		(at 189.23 254 0)
-		(fields_autoplaced yes)
 		(effects
 			(font
@@
 	(label "CC1"
 		(at 189.23 251.46 0)
-		(fields_autoplaced yes)
 		(effects
 			(font
@@
 	(label "PWR_EN"
 		(at 361.95 168.91 0)
-		(fields_autoplaced yes)
 		(effects
 			(font
@@
 	(label "PWR_C_D-"
 		(at 189.23 261.62 0)
-		(fields_autoplaced yes)
 		(effects
 			(font
@@
 		(shape output)
 		(at 341.63 300.99 180)
-		(fields_autoplaced yes)
 		(effects
 			(font
@@
 		(shape input)
 		(at 328.93 200.66 180)
-		(fields_autoplaced yes)
 		(effects
 			(font
@@
 		(shape input)
 		(at 328.93 213.36 180)
-		(fields_autoplaced yes)
 		(effects
 			(font
@@
 		(shape output)
 		(at 379.73 300.99 180)
-		(fields_autoplaced yes)
 		(effects
 			(font
